File: pcb_lm3424/pcb_lm3424.kicad_pcb (KiCad board)
At the start: 2 copper layers, 49 x 30 mm, 54 parts, among them J1 PWM, J2 VIN, J3 SYNC, J4 GND, J5 NTC, J6 NTC, J7 +, J8 –, Q1 2N7002, Q2 PSMN025-80YLX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

Commit message: Gerber settings
Other:
- board text added: "constant-current-LED-driver"
Changed lines of the file:
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@@
-(kicad_pcb (version 20171130) (host pcbnew 5.1.2-1.fc30)
+(kicad_pcb (version 20171130) (host pcbnew 5.1.4-1.fc30)
   (general
     (thickness 1.6)
-    (drawings 25)
+    (drawings 26)
     (tracks 368)
     (zones 0)
@@
     (pad_to_mask_clearance 0.025)
     (solder_mask_min_width 0.1)
-    (aux_axis_origin 0 0)
+    (aux_axis_origin 100 120)
+    (grid_origin 100 120)
     (visible_elements FFFFFF7F)
     (pcbplotparams
       (layerselection 0x010fc_ffffffff)
-      (usegerberextensions false)
+      (usegerberextensions true)
       (usegerberattributes false)
       (usegerberadvancedattributes false)
@@
       (outputformat 1)
       (mirror false)
-      (drillshape 1)
+      (drillshape 0)
       (scaleselection 1)
-      (outputdirectory ""))
+      (outputdirectory "gerber_lm3424/"))
   )
   (net 0 "")
@@
       (rotate (xyz 0 0 0))
     )
+  )
+  (gr_text "constant-current-LED-driver " (at 124.25 121) (layer B.Mask)
+    (effects (font (size 1 1) (thickness 0.15)) (justify mirror))
   )
   (gr_line (start 122.3 149.8) (end 119.9 149.8) (layer F.SilkS) (width 0.12))
@@
     (polygon
       (pts
-        (xy 98 118) (xy 151 118) (xy 151 152) (xy 98 152)
+        (xy 100 120) (xy 113 120) (xy 113 121.75) (xy 136 121.75) (xy 136 120)
+        (xy 149 120) (xy 149 150) (xy 100 150)
       )
     )
